File: BMS_USBC_2S.kicad_sch (KiCad schematic)
At the start: 30 parts

Commit message: Add pcb and power output connector
Parts:
- added J4: Conn_01x02, Connector_PinSocket_2.54mm:PinSocket_1x02_P2.54mm_Vertical, symbol Connector:Conn_01x02_Female
- C1, C2, C3, C4, C5, C6, C7, C8, C9: renamed from C?; footprint (none) -> Capacitor_SMD:C_0805_2012Metric
- D1, D3: renamed from D?; footprint (none) -> LED_SMD:LED_0603_1608Metric
- D2: renamed from D?; footprint (none) -> Diode_SMD:D_SMA-SMB_Universal_Handsoldering; LCSC (none) -> C3011099
- IC1, IC2: renamed from IC?; footprint SOT23-6 -> Footprint:SOT23-6
- J1: renamed from J?; footprint (none) -> Connector_USB:USB_C_Receptacle_Amphenol_12401610E4-2A
- J2: renamed from J?; footprint (none) -> Connector_PinSocket_2.54mm:PinSocket_1x02_P2.54mm_Vertical
- J3: renamed from J?; footprint (none) -> Connector_PinHeader_2.54mm:PinHeader_1x03_P2.54mm_Vertical
- L1: renamed from L?; footprint (none) -> Footprint:MDA7030-220M; LCSC (none) -> C2847487
- Q1, Q2: renamed from Q?; footprint SOP65P640X120-8N -> Footprint:SOP65P640X120-8N; LCSC (none) -> C2830320
- R1, R2, R3, R4, R5, R6, R7, R8, R9: renamed from R?; footprint (none) -> Resistor_SMD:R_0805_2012Metric
- U1: renamed from U?; footprint (none) -> Footprint:QFN-16_EP_3.9x3.9_Pitch0.65mm
Connections:
- net BATT_1+: now also J4.2 (Pin_2)
- net GND: now also J4.1 (Pin_1)
Other:
- note added: "Balance Plug"
- note added: "Safe Output"
- note added: "THM1 10K NTC Thermistor"
- moved on the sheet: C1, C2, C3, C4, C5, C6, C7, D1, D2, D3, J1, J2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
